Commit message: Modified for use with Sawyer

File: kinect_v2/urdf/kinect_v2.urdf.xacro (robot description, xacro)
@@ -19,8 +19,8 @@
                 <origin xyz="0 0 0" rpy="0 0 0" />
                 <geometry>
-                    <mesh filename="package://dhbot_description/meshes/kinect2.STL" />
+                    <mesh filename="package://kinect_v2/meshes/kinect2.STL" />
                 </geometry>
                 <material name="">
-                    <color rgba="0.5 0.5 0.5 1" />
+                    <!--color rgba="0.01 0.01 0.01 1" /-->
                 </material>
             </visual>
@@ -28,5 +28,5 @@
                 <origin xyz="0 0 0" rpy="0 0 0" />
                 <geometry>
-                    <mesh filename="package://dhbot_description/meshes/kinect2.STL" />
+                    <mesh filename="package://kinect_v2/meshes/kinect2.STL" />
                 </geometry>
             </collision>
@@ -64,4 +64,7 @@
         <!-- gazebo extensions -->
         <xacro:kinect2_ir_gazebo link_name="kinect2_ir_link" frame_name="kinect2_ir_optical_frame" camera_name="kinect_V2" />
+	<gazebo reference="kinect2_base_link">
+        <material>Gazebo/FlatBlack</material>
+        </gazebo>
     </xacro:macro>
 </robot>

File: kinect_v2/urdf/kinect_v2_standalong.urdf.xacro (robot description, xacro)
@@ -4,6 +4,9 @@
      <link name="root"/>
     <xacro:kinect_v2  parent="root">
-        <origin xyz="0 0 0"
-                rpy="0 0 0" />
+        <origin xyz="0 0.1 1.50"
+                rpy="0 0.785398 0" />
     </xacro:kinect_v2>
+    <gazebo>
+    <static>true</static>
+    </gazebo>
 </robot>
