Commit message: Many changes

File: kinect_v2/urdf/kinect_v2.gazebo.xacro (robot description, xacro)
@@ -2,5 +2,5 @@
 <robot xmlns:xacro="http://ros.org/wiki/xacro">
  <gazebo reference="kinect2_base_link">
-  <material>Gazebo/Grey</material>
+  <material>Gazebo/FlatBlack</material>
   </gazebo>
 <xacro:macro name="kinect2_ir_gazebo" params="link_name frame_name camera_name">
@@ -13,6 +13,6 @@
         <image>
           <format>L8</format>
-          <width>640</width>
-          <height>480</height>
+          <width>1280</width>	<!-- 1920 -->
+          <height>800</height>	<!-- 1080 -->
         </image>
         <clip>
@@ -57,6 +57,6 @@
         <image>
           <format>B8G8R8</format>
-          <width>640</width>
-          <height>480</height>
+          <width>1280</width>	<!-- 1920 -->
+          <height>800</height>	<!-- 1080 -->
         </image>
         <clip>

File: kinect_v2/urdf/kinect_v2.urdf.xacro (robot description, xacro)
@@ -22,5 +22,5 @@
                 </geometry>
                 <material name="">
-                    <!--color rgba="0.01 0.01 0.01 1" /-->
+                    <color rgba="0.5 0.5 0.5 1" />
                 </material>
             </visual>
@@ -64,7 +64,4 @@
         <!-- gazebo extensions -->
         <xacro:kinect2_ir_gazebo link_name="kinect2_ir_link" frame_name="kinect2_ir_optical_frame" camera_name="kinect_V2" />
-	<gazebo reference="kinect2_base_link">
-        <material>Gazebo/FlatBlack</material>
-        </gazebo>
     </xacro:macro>
 </robot>

File: kinect_v2/urdf/kinect_v2_standalong.urdf.xacro (robot description, xacro)
@@ -4,6 +4,6 @@
      <link name="root"/>
     <xacro:kinect_v2  parent="root">
-        <origin xyz="0 0.1 1.50"
-                rpy="0 0.785398 0" />
+        <origin xyz="2.2 0 1.6"
+                rpy="0 0.349066 3.1415" /> <!-- 2.2 0 1.6 0 0.349066 3.1415 -->
     </xacro:kinect_v2>
     <gazebo>
